File: picdiv_board_v3.kicad_pcb (KiCad board)
At the start: 2 copper layers, 75 x 100 mm, 81 parts, among them J1 DC-Input, J10 PPS_B, J101 MountingHole_M2.5, J102 Conn_Coaxial, J103 Conn_Coaxial, J104 MountingHole_M2.5, J105 Conn_01x06, J106 PPS_A, J107 PPS_A, J14 TEST_1PPS, J4 SYNC, J6 PPS_B, J8 SYNC, Q1 Q_PNP_BEC, Q2 Q_PNP_BEC, SW101 SW_DIP_x03, U1 LT1963AxST-3.3, U103 LT1963AEQ, U104 LTC6993xS6-1, U105 IDT5PB1108, U2 LT1963AxST-3.3, U3 PIC12F675, U6 IDT5PB1108

Commit message: Ignore Backups
Other:
- board text removed: "multi-cb pricing as of 2018-08 75x100, 2-sided, ENIG, top-silk ca 24eur/pcs for two"
