File: picdiv_board_v3.kicad_sch (KiCad schematic)
At the start: 81 parts, among them J1 DC-Input, J10 PPS_B, J101 MountingHole_M2.5, J102 Conn_Coaxial, J103 Conn_Coaxial, J104 MountingHole_M2.5, J105 Conn_01x06, J106 PPS_A, J107 PPS_A, J14 TEST_1PPS, J4 SYNC, J6 PPS_B, J8 SYNC, Q1 Q_PNP_BEC, Q2 Q_PNP_BEC, SW101 SW_DIP_x03, U1 LT1963AxST-3.3, U103 LT1963AEQ, U104 LTC6993xS6-1, U105 IDT5PB1108, U2 LT1963AxST-3.3, U3 PIC12F675, U6 IDT5PB1108

Commit message: Ignore Backups
Parts:
- removed C1, C13: 10n, Capacitor_SMD:C_0805_2012Metric, symbol Device:C
- removed C12, C17, C2, C20: 100n, Capacitor_SMD:C_0805_2012Metric, symbol Device:C
- removed C8: C_Trim, Capacitor_SMD:C_Trimmer_Murata_TZB4-A, symbol Device:C_Trim
- removed CLK101: TEST_CLK, TestPoint:TestPoint_2Pads_Pitch2.54mm_Drill0.8mm, symbol Connector:TestPoint_2Pole
- removed J10: PPS_B, Connector_Coaxial:BNC_Amphenol_B6252HB-NPP3G-50_Horizontal, symbol Connector:Conn_Coaxial
- removed J102: Conn_Coaxial, Connector_Coaxial:BNC_Amphenol_B6252HB-NPP3G-50_Horizontal, symbol Connector:Conn_Coaxial
- removed J103: Conn_Coaxial, Connector_Coaxial:SMA_Molex_73251-2200_Horizontal, symbol Connector:Conn_Coaxial
- removed J6: PPS_B, Connector_Coaxial:SMA_Molex_73251-2200_Horizontal, symbol Connector:Conn_Coaxial
- removed L1: 100u (1210), Inductor_SMD:L_1210_3225Metric, symbol Device:L
- removed L4: 2u2, Inductor_SMD:L_0805_2012Metric, symbol Device:L
- removed Q1, Q2: Q_PNP_BEC, TO_SOT_Packages_SMD:SOT-23, symbol Device:Q_PNP_BEC
- removed R1: 49R9, Resistor_SMD:R_0805_2012Metric, symbol Device:R
- removed R2, R7: 3k3, Resistor_SMD:R_0805_2012Metric, symbol Device:R
- removed R3, R8: 6k8, Resistor_SMD:R_0805_2012Metric, symbol Device:R
- removed R4, R5: 220R, Resistor_SMD:R_0805_2012Metric, symbol Device:R
- removed R6: 270R, Resistor_SMD:R_0805_2012Metric, symbol Device:R
- removed U6: IDT5PB1108, Package_SO:TSSOP-16_4.4x5mm_P0.65mm, symbol Interface:5PB1108PGxx
- added U4: ~, Oscilator_Local:OSC5A2B02, symbol Oscillator_Local:OSC5AB02
Connections:
- net GND: now also U4.2 (GND)
- net PPS: now also U4.1 (Out)
- no-connect marks 9 -> 5
Other:
- note removed: "10MHz sinewave input XX dBm to YY dBm (to be measured)"
- note removed: "10MHz square-wave clock for PIC"
- note removed: "4.07VDC with 6VCC"
- note removed: "800-2895-5-ND"
- note removed: "Q1 and Q2 2N3906 MMBT3906-FDICT-ND SOT23-3"
- note removed: "Sine-to-square converter circuit: TADD-2-mini: https://www.tapr.org/~{n8ur/T2_Mini_Manual.pdf} Wenzel: http://www.wenzel.com/documents/waveform.html,"
- moved on the sheet: C10, D4, J14, R10, R15, R16, R18, U104
