File: OXCO.kicad_sch (KiCad schematic)
At the start: 21 parts, among them U7 LT1963AEQ, U8 ADR4540

Commit message: More layout, mostly around Vadg
Parts:
- removed C26: 100nF, Capacitor_SMD:C_0402_1005Metric_Pad0.74x0.62mm_HandSolder, symbol Device:C
- C20: renamed from C21; value 10u -> 10µF
- D6: LCSC (none) -> C2297
- renumbered C20 to C21
Changed lines of the file:
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@@
 	(wire
 		(pts
-			(xy 138.43 99.06) (xy 138.43 101.6)
-		)
-		(stroke
-			(width 0)
-			(type default)
-		)
-	)
-	(wire
-		(pts
 			(xy 43.18 59.69) (xy 43.18 66.04)
 		)
@@
 		(on_board yes)
 		(dnp no)
-		(property "Reference" "C21"
+		(property "Reference" "C20"
 			(at 89.535 133.35 0)
 			(effects
@@
 			)
 		)
-		(property "Value" "10u"
+		(property "Value" "10µF"
 			(at 89.535 128.27 0)
 			(effects
@@
 			(project "picdiv_board_v3"
 				(path "/eba36321-b5f3-4bd6-a805-57b9b2ee447e/e769b68a-585d-4de6-8d1e-4dcee65d99b9"
-					(reference "C21")
+					(reference "C20")
 					(unit 1)
 				)
@@
 		(dnp no)
 		(fields_autoplaced yes)
-		(property "Reference" "C20"
+		(property "Reference" "C21"
 			(at 83.82 74.9299 0)
 			(effects
@@
 			(project "picdiv_board_v3"
 				(path "/eba36321-b5f3-4bd6-a805-57b9b2ee447e/e769b68a-585d-4de6-8d1e-4dcee65d99b9"
-					(reference "C20")
+					(reference "C21")
 					(unit 1)
 				)
@@
 	(symbol
 		(lib_id "power:GND")
-		(at 138.43 101.6 0)
-		(unit 1)
-		(exclude_from_sim no)
-		(in_bom yes)
-		(on_board yes)
-		(dnp no)
-		(fields_autoplaced yes)
-		(property "Reference" "#PWR023"
-			(at 138.43 107.95 0)
-			(effects
-				(font
-					(size 1.27 1.27)
-				)
-				(hide yes)
-			)
-		)
-		(property "Value" "GND"
-			(at 138.43 106.68 0)
-			(effects
-				(font
-					(size 1.27 1.27)
-				)
-			)
-		)
-		(property "Footprint" ""
-			(at 138.43 101.6 0)
-			(effects
-				(font
-					(size 1.27 1.27)
-				)
-				(hide yes)
-			)
-		)
-		(property "Datasheet" ""
-			(at 138.43 101.6 0)
-			(effects
-				(font
-					(size 1.27 1.27)
-				)
-				(hide yes)
-			)
-		)
-		(property "Description" "Power symbol creates a global label with name \"GND\" , ground"
-			(at 138.43 101.6 0)
-			(effects
-				(font
-					(size 1.27 1.27)
-				)
-				(hide yes)
-			)
-		)
-		(pin "1"
-		)
-		(instances
-			(project ""
-				(path "/eba36321-b5f3-4bd6-a805-57b9b2ee447e/e769b68a-585d-4de6-8d1e-4dcee65d99b9"
-					(reference "#PWR023")
-					(unit 1)
-				)
-			)
-		)
-	)
-	(symbol
-		(lib_id "power:GND")
 		(at 59.69 137.16 0)
 		(unit 1)
@@
 	)
 	(symbol
-		(lib_id "Device:C")
-		(at 138.43 95.25 0)
-		(unit 1)
-		(exclude_from_sim no)
-		(in_bom yes)
-		(on_board yes)
-		(dnp no)
-		(fields_autoplaced yes)
-		(property "Reference" "C26"
-			(at 142.24 93.9799 0)
-			(effects
-				(font
-					(size 1.27 1.27)
-				)
-				(justify left)
-			)
-		)
-		(property "Value" "100nF"
-			(at 142.24 96.5199 0)
-			(effects
-				(font
-					(size 1.27 1.27)
-				)
-				(justify left)
-			)
-		)
-		(property "Footprint" "Capacitor_SMD:C_0402_1005Metric_Pad0.74x0.62mm_HandSolder"
-			(at 139.3952 99.06 0)
-			(effects
-				(font
-					(size 1.27 1.27)
-				)
-				(hide yes)
-			)
-		)
-		(property "Datasheet" "~"
-			(at 138.43 95.25 0)
-			(effects
-				(font
-					(size 1.27 1.27)
-				)
-				(hide yes)
-			)
-		)
-		(property "Description" "Unpolarized capacitor"
-			(at 138.43 95.25 0)
-			(effects
-				(font
-					(size 1.27 1.27)
-				)
-				(hide yes)
-			)
-		)
-		(property "LCSC" "C1525"
-			(at 138.43 95.25 0)
-			(effects
-				(font
-					(size 1.27 1.27)
-				)
-				(hide yes)
-			)
-		)
-		(property "MPN" "CL05B104KO5NNNC "
-			(at 138.43 95.25 0)
-			(effects
-				(font
-					(size 1.27 1.27)
-				)
-				(hide yes)
-			)
-		)
-		(pin "2"
-		)
-		(pin "1"
-		)
-		(instances
-			(project "picdiv_board_v4AF"
-				(path "/eba36321-b5f3-4bd6-a805-57b9b2ee447e/e769b68a-585d-4de6-8d1e-4dcee65d99b9"
-					(reference "C26")
-					(unit 1)
-				)
-			)
-		)
-	)
-	(symbol
 		(lib_id "power:GND")
 		(at 41.91 135.89 0)
@@
 			(at 81.28 130.81 0)
 			(effects
+				(font
+					(size 1.27 1.27)
+				)
+				(hide yes)
+			)
+		)
+		(property "MPN" ""
+			(at 81.28 130.81 0)
+			(effects
+				(font
+					(size 1.27 1.27)
+				)
+				(hide yes)
+			)
+		)
+		(property "LCSC" "C2297 "
+			(at 81.28 130.81 0)
+			(effects

Commit message: Highlight a DRC error
Needs  more work.
Changed lines of the file:
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@@
 (kicad_sch
-	(version 20231120)
+	(version 20250114)
 	(generator "eeschema")
-	(generator_version "8.0")
+	(generator_version "9.0")
 	(paper "A4")
+	(text "ADR4540ARZ 4ppm/°C"
+		(exclude_from_sim no)
+		(at 68.072 52.07 0)
+		(effects
+			(font
+				(size 1.27 1.27)
+			)
+		)
+	)
+	(text "ADR4540BRZ 2ppm/°C"
+		(exclude_from_sim no)
+		(at 68.326 55.118 0)
+		(effects
+			(font
+				(size 1.27 1.27)
+			)
+		)
+	)
+	(text "1.365V"
+		(exclude_from_sim no)
+		(at 130.81 96.774 0)
+		(effects
+			(font
+				(size 1.27 1.27)
+			)
+		)
+	)
+	(text "LT1963AEQ"
+		(exclude_from_sim no)
+		(at 53.848 119.634 0)
+		(effects
+			(font
+				(size 1.524 1.524)
+			)
+			(justify left bottom)
+		)
+	)
+	(text "4.096V"
+		(exclude_from_sim no)
+		(at 86.36 68.072 0)
+		(effects
+			(font
+				(size 1.27 1.27)
+			)
+		)
+	)
+	(text "Vishay 1280G has similar footprint as Bourns 3005P\n and 3006P. Possible to layout so all three fit. "
+		(exclude_from_sim no)
+		(at 127 110.49 0)
+		(effects
+			(font
+				(size 1.27 1.27)
+			)
+		)
+	)
+	(text "Bourns 3006P-1-202 100pm  3/4\"  £1.62\nBourns 3005P-1-202 50ppm  3/4\"  £18.50 (Mouser)\n"
+		(exclude_from_sim no)
+		(at 60.96 94.234 0)
+		(effects
+			(font
+				(face "Arial")
+				(size 1.27 1.27)
+			)
+		)
+	)
+	(text "3.000V"
+		(exclude_from_sim no)
+		(at 137.922 82.296 0)
+		(effects
+			(font
+				(size 1.27 1.27)
+			)
+		)
+	)
+	(text "OSC5AB02"
+		(exclude_from_sim no)
+		(at 186.182 62.738 0)
+		(effects
+			(font
+				(size 1.27 1.27)
+			)
+		)
+	)
+	(text "Vishay 1280G  10%, ±15ppm Foil £24.48 (Mouser) "
+		(exclude_from_sim no)
+		(at 60.706 97.536 0)
+		(effects
+			(font
+				(size 1.27 1.27)
+			)
+		)
+	)
+	(text "5VDC for OXCO"
+		(exclude_from_sim no)
+		(at 72.39 124.46 0)
+		(effects
+			(font
+				(size 1.27 1.27)
+			)
+			(justify left bottom)
+		)
+	)
 	(junction
 		(at 81.28 146.05)
@@
 	)
 	(junction
-		(at 138.43 90.17)
-		(diameter 0)
-		(color 0 0 0 0)
-	)
-	(junction
 		(at 226.06 57.15)
 		(diameter 0)
@@
 	(wire
 		(pts
-			(xy 129.54 90.17) (xy 138.43 90.17)
+			(xy 129.54 90.17) (xy 143.51 90.17)
 		)
 		(stroke
@@
 	(wire
 		(pts
-			(xy 138.43 90.17) (xy 138.43 91.44)
-		)
-		(stroke
-			(width 0)
-			(type default)
-		)
-	)
-	(wire
-		(pts
 			(xy 80.01 69.85) (xy 92.71 69.85)
 		)
@@
 	(wire
 		(pts
-			(xy 138.43 90.17) (xy 143.51 90.17)
-		)
-		(stroke
-			(width 0)
-			(type default)
-		)
-	)
-	(wire
-		(pts
 			(xy 105.41 99.06) (xy 125.73 99.06)
 		)
@@
 		)
 	)
-	(text "ADR4540ARZ 4ppm/°C"
-		(exclude_from_sim no)
-		(at 68.072 52.07 0)
-		(effects
-			(font
-				(size 1.27 1.27)
-			)
-		)
-	)
-	(text "ADR4540BRZ 2ppm/°C"
-		(exclude_from_sim no)
-		(at 68.326 55.118 0)
-		(effects
-			(font
-				(size 1.27 1.27)
-			)
-		)
-	)
-	(text "1.365V"
-		(exclude_from_sim no)
-		(at 130.81 96.774 0)
-		(effects
-			(font
-				(size 1.27 1.27)
-			)
-		)
-	)
-	(text "LT1963AEQ"
-		(exclude_from_sim no)
-		(at 53.848 119.634 0)
-		(effects
-			(font
-				(size 1.524 1.524)
-			)
-			(justify left bottom)
-		)
-	)
-	(text "4.096V"
-		(exclude_from_sim no)
-		(at 86.36 68.072 0)
-		(effects
-			(font
-				(size 1.27 1.27)
-			)
-		)
-	)
-	(text "Vishay 1280G has similar footprint as Bourns 3005P\n and 3006P. Possible to layout so all three fit. "
-		(exclude_from_sim no)
-		(at 127 110.49 0)
-		(effects
-			(font
-				(size 1.27 1.27)
-			)
-		)
-	)
-	(text "Bourns 3006P-1-202 100pm  3/4\"  £1.62\nBourns 3005P-1-202 50ppm  3/4\"  £18.50 (Mouser)\n"
-		(exclude_from_sim no)
-		(at 60.96 94.234 0)
-		(effects
-			(font
-				(face "Arial")
-				(size 1.27 1.27)
-			)
-		)
-	)
-	(text "3.000V"
-		(exclude_from_sim no)
-		(at 137.922 82.296 0)
-		(effects
-			(font
-				(size 1.27 1.27)
-			)
-		)
-	)
-	(text "OSC5AB02"
-		(exclude_from_sim no)
-		(at 186.182 62.738 0)
-		(effects
-			(font
-				(size 1.27 1.27)
-			)
-		)
-	)
-	(text "Vishay 1280G  10%, ±15ppm Foil £24.48 (Mouser) "
-		(exclude_from_sim no)
-		(at 60.706 97.536 0)
-		(effects
-			(font
-				(size 1.27 1.27)
-			)
-		)
-	)
-	(text "5VDC for OXCO"
-		(exclude_from_sim no)
-		(at 72.39 124.46 0)
-		(effects
-			(font
-				(size 1.27 1.27)
-			)
-			(justify left bottom)
-		)
-	)
 	(global_label "LDO_IN"
 		(shape input)
@@
 			)
 		)
-		(property "Description" "1% 100ppm - Basic part"
+		(property "Description" "Resistor"
 			(at 74.93 140.97 0)
 			(effects
@@
 			)
 		)
-		(property "Datasheet" "https://www.bourns.com/docs/product-datasheets/3006.pdf?sfvrsn=47e86352_10"
+		(property "Datasheet" "~"
 			(at 125.73 90.17 0)
 			(effects
@@
 			)
 		)
-		(property "Description" "2.15kΩ ±25ppm/℃ ±0.1%"
+		(property "Description" "Resistor"
 			(at 74.93 130.81 0)
 			(effects
@@
 			(at 81.28 130.81 0)
 			(effects
+				(font
+					(size 1.27 1.27)
+				)
+				(hide yes)
+			)
+		)
+		(property "Sim.Pins" "1=K 2=A"
+			(at 81.28 130.81 0)
+			(effects
